File: kicad/SSDV3.kicad_pcb (KiCad board)
At the start: 4 copper layers, 58.4 x 28.8 mm, 72 parts, among them J1 SolderPad, J2 SolderPad, J3 SolderPad, J4 SolderPad, J5 SolderPad, J6 SolderPad, J7 SolderPad_01x02, J8 SolderPad_1x03, Q1 CSD19537Q3, Q2 CSD19537Q3, Q3 BSZ096N10LS5, U1 LM5050-1, U2 LM5146RGYR

Commit message: Officially now the SSDV3
Parts:
- U2: footprint LM5146RGYR:RGY0020B-MFG -> ul_LM5146RGYR:RGY0020B-MFG-ThermalVias
Changed lines of the file:
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@@
 	(title_block
 		(title "Super Step Down V3")
-		(date "2025-10-19")
+		(date "2025-10-20")
 		(rev "C")
 		(company "UBCO Aerospace [Julian Joaquin]")
@@
 		)
 		(property "Value" "SolderPad_1x03"
-			(at 0 2.54 0)
+			(at 0.96 4.15 0)
 			(layer "F.Fab")
 			(effects
@@
 		)
 		(fp_text user "${REFERENCE}"
-			(at 0 0 0)
+			(at 1.96 -0.05 0)
 			(layer "F.Fab")
 			(effects
@@
 		)
 		(property "Value" "BSZ096N10LS5"
-			(at 0 3 270)
+			(at 1.654083 2.45 270)
 			(unlocked yes)
 			(layer "F.Fab")
@@
 		)
 		(property "Value" "CSD19537Q3"
-			(at 0 2.5 0)
+			(at 6.65 -1.8 0)
 			(unlocked yes)
 			(layer "F.Fab")
@@
 		)
 	)
-	(footprint "LM5146RGYR:RGY0020B-MFG"
+	(footprint "ul_LM5146RGYR:RGY0020B-MFG-ThermalVias"
 		(layer "F.Cu")
 		(at 154.4 120.6 90)
@@
 		)
 		(property "Value" "CSD19537Q3"
-			(at 0 2.5 180)
+			(at 1.4 2.35 0)
 			(unlocked yes)
 			(layer "F.Fab")
