File: kicad/rpp.kicad_sch (KiCad schematic)
At the start: 13 parts, among them J1 SolderPad, J2 SolderPad, J3 SolderPad, J4 SolderPad, Q1 CSD19537Q3, U1 LM5050-1

Commit message: Layout tweaks, added copyright notice
Other:
- company: Julian Joaquin -> Author: Julian Joaquin
Changed lines of the file:
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@@
 	(title_block
 		(title "Super Step Down V3")
-		(date "2025-11-04")
+		(date "2025-11-08")
 		(rev "D")
-		(company "Julian Joaquin")
-		(comment 1 "A 12S battery eliminator circuit (BEC) for UAS applications.")
+		(company "Author: Julian Joaquin")
+		(comment 1 "Licensed under CERN-OHL-W version 2")
+		(comment 2 "Copyright © Julian Joaquin, 2025")
+		(comment 4 "A 12S battery eliminator circuit (BEC) for UAS applications.")
 	)
 	(text "Reverse polarity protection"
