File: kicad/SSDV3.kicad_sch (KiCad schematic)
At the start: 8 parts, among them J3 Conn_01x02_MountingPin, J4 Conn_01x03_MountingPin

Commit message: Initial layout for version 4
Parts:
- removed H1, H2, H3: MountingHole, MountingHole:ToolingHole_1.152mm, symbol Mechanical:MountingHole
- J3: value Conn_01x02_MountingPin -> SM02B-GHS-TB; footprint Connector_JST:JST_GH_SM02B-GHS-TB_1x02-1MP_P1.25mm_Horizontal -> Connector_JST:JST_GH_BM02B-GHS-TBT_1x02-1MP_P1.25mm_Vertical
- J4: value Conn_01x03_MountingPin -> SM03B-GHS-TB; footprint Connector_JST:JST_GH_SM03B-GHS-TB_1x03-1MP_P1.25mm_Horizontal -> Connector_JST:JST_GH_BM03B-GHS-TBT_1x03-1MP_P1.25mm_Vertical
