File: kicad/buck_converter.kicad_sch (KiCad schematic)
At the start: 51 parts, among them J1 XT30U-M, J2 XT30U-F, Q1 BSZ146N10LS5ATMA1, Q2 BSZ146N10LS5ATMA1, U1 LM5146

Commit message: Initial layout for version 4
Parts:
- removed C10, C11: 100nF, Capacitor_SMD:C_0603_1608Metric, symbol Device:C
- removed C12: 2.2uF, Capacitor_SMD:C_0805_2012Metric, symbol Device:C
- removed C13: 47nF, Capacitor_SMD:C_0603_1608Metric, symbol Device:C
- removed C14, C15: 2.2nF, Capacitor_SMD:C_0603_1608Metric, symbol Device:C
- removed C17: 100nF, Capacitor_SMD:C_0603_1608Metric, symbol Device:C_Small
- removed C18: 12pF, Capacitor_SMD:C_0603_1608Metric, symbol Device:C_Small
- removed C23: 22uF, Capacitor_SMD:C_1206_3216Metric, symbol Device:C
- removed C3: 4.7uF, Capacitor_SMD:C_1206_3216Metric, symbol Device:C
- removed JP1: 7.4V, Jumper:SolderJumper-2_P1.3mm_Open_TrianglePad1.0x1.5mm, symbol Jumper:Jumper_2_Open
- removed JP2: 9.6V, Jumper:SolderJumper-2_P1.3mm_Open_TrianglePad1.0x1.5mm, symbol Jumper:Jumper_2_Open
- removed Q1: BSZ146N10LS5ATMA1, Package_SON_JJ:Infineon_PG-TSDSON-8-26_3.3x3.3mm_P0.65mm_ThermalVias-D0.3mm, symbol Julian_Symbols:BSZ096N10LS5
- removed Q2: BSZ146N10LS5ATMA1, Package_SON_JJ:Infineon_PG-TSDSON-8-26_3.3x3.3mm_P0.65mm, symbol Julian_Symbols:BSZ096N10LS5
- removed R14: 2.2, Resistor_SMD:R_0603_1608Metric, symbol Device:R_Small_US
- removed R15: 430, Resistor_SMD:R_0603_1608Metric, symbol Device:R_Small_US
- removed R4: 20k, Resistor_SMD:R_0603_1608Metric, symbol Device:R_Small_US
- removed R6, R9: 20k, Resistor_SMD:R_0603_1608Metric, symbol Device:R_US
- removed R8: 1k, Resistor_SMD:R_0603_1608Metric, symbol Device:R_US
- removed U1: LM5146, Package_QFN_JJ:Texas_RGY0020B_EP_3.5x4.5mm_P0.5mm_ThermalVias-D0.3mm, symbol Julian_Symbols:LM5146RGYR
- added C1: 100nF, Capacitor_SMD:C_0402_1005Metric, symbol Device:C
- added C12, C15, C9: 100nF, Capacitor_SMD:C_0402_1005Metric, symbol Device:C_Small
- added C14: 2.2uF, Capacitor_SMD:C_0603_1608Metric, symbol Device:C_Small
- added C17, C18, C24, C27: 10nF, Capacitor_SMD:C_0402_1005Metric, symbol Device:C
- added C19: 390pF, Capacitor_SMD:C_0402_1005Metric, symbol Device:C_Small
- added C2: 4.7nF, Capacitor_SMD:C_0603_1608Metric_Pad1.08x0.95mm_HandSolder, symbol Device:C
- added C25, C26, C28, C30, C36, C37, C38, C39, C40: 22uF, Capacitor_SMD:C_0805_2012Metric, symbol Device:C
- added C31, C33, C34: 220nF, Capacitor_SMD:C_0603_1608Metric, symbol Device:C
- added C35: 47uF, ul_16TQC47MYFB:CAP_TQC_B2_PAN, symbol Device:C_Polarized_US
- added C5: 2.2uF, Capacitor_SMD:C_0603_1608Metric, symbol Device:C
- added C7: 4.7uF, Capacitor_SMD:C_1206_3216Metric_Pad1.33x1.80mm_HandSolder, symbol Device:C
- added Q1: LMG2100R044, ul_LMG2100R044RARR:RAR0016B-MFG, symbol Julian_Symbols:LMG2100R044
- added R1: 7.5k, Resistor_SMD:R_0603_1608Metric_Pad0.98x0.95mm_HandSolder, symbol Device:R_US
- added R15: 0, Resistor_SMD:R_0603_1608Metric_Pad0.98x0.95mm_HandSolder, symbol Device:R_US
- added R4: 4.99k, Resistor_SMD:R_0603_1608Metric_Pad0.98x0.95mm_HandSolder, symbol Device:R_US
- added R8: 2, Resistor_SMD:R_0402_1005Metric_Pad0.72x0.64mm_HandSolder, symbol Device:R_Small_US
- added R9: 510, Resistor_SMD:R_0402_1005Metric, symbol Device:R_Small_US
- added U1: LM5148, Package_QFN_JJ:Texas_RGY0024F_EP_3.5x5.5mm_P0.5_ThermalVias-D0.2mm, symbol Julian_Symbols:LM5148RGYR
- C10: renamed from C6; footprint Capacitor_SMD:C_1206_3216Metric -> Capacitor_SMD:C_1206_3216Metric_Pad1.33x1.80mm_HandSolder
- C11: renamed from C7; footprint Capacitor_SMD:C_1206_3216Metric -> Capacitor_SMD:C_1206_3216Metric_Pad1.33x1.80mm_HandSolder
- C13: renamed from C8; footprint Capacitor_SMD:C_1206_3216Metric -> Capacitor_SMD:C_1206_3216Metric_Pad1.33x1.80mm_HandSolder
- C16: value 10pF -> 10nF; footprint Capacitor_SMD:C_0603_1608Metric -> Capacitor_SMD:C_0402_1005Metric; LCSC PN C1634 -> C527014; Manufacturer Panasonic -> YAGEO; Part Number CL10C100JB8NNNC -> CC0402KRX7R0BB103; Part Type Basic -> Extended; Tolerance 5% -> 10%; Voltage 50V -> 100V
- C20, C21, C22: value 22uF -> 10nF; footprint Capacitor_SMD:C_1206_3216Metric -> Capacitor_SMD:C_0402_1005Metric; ESR 3.4mΩ -> (none); LCSC PN C5272872 -> C527014; Manufacturer Murata Electronics -> YAGEO; Part Number GRM31CC71E226ME15L -> CC0402KRX7R0BB103; Voltage 25V -> 100V
- C23: renamed from C19; footprint Capacitor_SMD:C_1206_3216Metric -> Capacitor_SMD:C_0805_2012Metric; ESR 3.4mΩ -> 2mΩ; LCSC PN C5272872 -> C86816; Part Number GRM31CC71E226ME15L -> GRM21BR61E226ME44L; Tolerance 10% -> 20%
- C29: renamed from C9; value 100nF -> 220nF; LCSC PN C113803 -> C7300906; Manufacturer YAGEO -> Taiyo Yuden; Part Number CC0603KRX7R0BB104 -> MCASH168SC7224KTCA01
- C32: renamed from C24; value 100uF -> 47uF; footprint Capacitor_Tantalum_SMD:CP_EIA-7343-20_Kemet-V_HandSolder -> ul_16TQC47MYFB:CAP_TQC_B2_PAN; ESR 18mΩ -> 43mΩ; LCSC PN C696814 -> C4987277; Part Number T521D107M025ATE040 -> 16TQC47MYFB; Voltage 25V -> 16V
- C4: value 4.7uF -> 68pF; footprint Capacitor_SMD:C_1206_3216Metric -> Capacitor_SMD:C_0603_1608Metric_Pad1.08x0.95mm_HandSolder; ESR 2mΩ -> (none); FT Rotation Offset 0 -> (none); LCSC PN C3864744 -> C28262; Manufacturer Murata Electronics -> Samsung Electro-Mechanics; Part Number GRJ31CZ72A475KE01L -> CL10C680JB8NNNC; Part Type Extended -> Basic; Tolerance 10% -> (none); Voltage 100V -> (none)
- C6: renamed from C2; value 100nF -> 220nF; LCSC PN C113803 -> C7300906; Manufacturer YAGEO -> Taiyo Yuden; Part Number CC0603KRX7R0BB104 -> MCASH168SC7224KTCA01
- C8: renamed from C5; footprint Capacitor_SMD:C_1206_3216Metric -> Capacitor_SMD:C_1206_3216Metric_Pad1.33x1.80mm_HandSolder
- D1: LCSC PN (none) -> C19077594; Manufacturer (none) -> R+O; Part Number (none) -> SMBJ64A; Part Type (none) -> Preferred Extended
- L1: footprint Inductor_SMD:L_Bourns_SRP1038C_10.0x10.0mm -> Inductor_SMD:L_Bourns_SRP1245A; ESR 15.5mΩ -> 8.4mΩ; LCSC PN C6949325 -> C780205; Manufacturer Pulse Electronics -> Bourns Incorperated; Part Number PA4342.472NLT -> SRP1265A-4R7M
- R10: value 6.8k -> 8m; footprint Resistor_SMD:R_0603_1608Metric -> Resistor_SMD:R_1206_3216Metric; FT Rotation Offset 0 -> (none); LCSC PN (none) -> C1720323; Manufacturer UNI-ROYAL -> YAGEO; Part Number (none) -> PE1206FRM470R008L; Part Type Basic -> Extended; Power 0.1W -> (none); Tolerance 1% -> (none); Voltage 75V -> (none)
- R11: value 6.81k -> 8m; footprint Resistor_SMD:R_0603_1608Metric -> Resistor_SMD:R_1206_3216Metric; FT Rotation Offset 0 -> (none); LCSC PN C861538 -> C1720323; Part Number RT0603BRD076K81L -> PE1206FRM470R008L; Power 0.1W -> (none); Tolerance 0.1% -> (none); Voltage 50V -> (none)
- R12: value 3.48k -> 20k; footprint Resistor_SMD:R_0603_1608Metric -> Resistor_SMD:R_0603_1608Metric_Pad0.98x0.95mm_HandSolder; FT Rotation Offset 0 -> (none); LCSC PN C423043 -> C4184; Part Number 0603WAD3481T5E -> 0603WAF2002T5E; Part Type Extended -> Basic; Power 0.1W -> (none); Tolerance 0.5% -> (none); Voltage 50V -> (none); now left out of the parts list
- R13: value 3.74k -> 1.43k; footprint Resistor_SMD:R_0603_1608Metric -> Resistor_SMD:R_0603_1608Metric_Pad0.98x0.95mm_HandSolder; FT Rotation Offset 0 -> (none); LCSC PN C849741 -> C861730; Part Number RT0603BRE073K74L -> RT0603BRE071K43L; Power 0.1W -> (none); Tolerance 0.1% -> (none); Voltage 75V -> (none)
- R2: value 150k -> 48.7k; FT Rotation Offset 0 -> (none); LCSC PN C22807 -> C165749; Manufacturer UNI-ROYAL -> YAGEO; Part Number 0603WAF1503T5E -> RC0603FR-0748K7L; Part Type Basic -> Extended; Power 0.1W -> (none); Tolerance 1% -> (none); Voltage 75V -> (none)
- R3: value 13k -> 200k; footprint Resistor_SMD:R_0603_1608Metric -> Resistor_SMD:R_0402_1005Metric; FT Rotation Offset 0 -> (none); LCSC PN C22797 -> C25764; Part Number 0603WAF1302T5E -> 0402WGF2003TCE; Power 0.1W -> (none); Tolerance 1% -> (none); Voltage 75V -> (none)
- R5: value 24k -> 41.2k; footprint Resistor_SMD:R_0603_1608Metric -> Resistor_SMD:R_0402_1005Metric; FT Rotation Offset 0 -> (none); LCSC PN C23352 -> C185416; Manufacturer UNI-ROYAL -> YAGEO; Part Number 0603WAF2402T5E -> RC0402FR-0741K2L; Part Type Basic -> Extended; Power 0.1W -> (none); Tolerance 1% -> (none); Voltage 75V -> (none)
- R6: renamed from R1; value 2.2 -> 2; footprint Resistor_SMD:R_0603_1608Metric -> Resistor_SMD:R_0402_1005Metric_Pad0.72x0.64mm_HandSolder; LCSC PN C22939 -> C270630; Part Number 0603WAF220KT5E -> 0402WGF200KTCE; Part Type Basic -> Extended
- R7: value 0 -> 48.7k; LCSC PN (none) -> C165749; Manufacturer (none) -> YAGEO; Part Number (none) -> RC0603FR-0748K7L; Part Type (none) -> Extended; now fitted; now in the parts list
- renumbered C1 to C3, R16 to R14
Connections:
- net COMP_RC1 is gone; now on net VOUT: R10.2
- net JP_CFG1 is gone; now on net VOUT: R11.2
- net SYNCIN is gone; now on net FB: R7.1
- net AGND: now also C4.2, NT1.1, R2.2, C1.2, C2.2, R4.2, U1.18 (PFM_SYNC), U1.7 (AGND); no longer NT1.2, R3.2, R7.2
- net COMP: now also C2.1, R1.1, U1.5 (EXTCOMP); no longer C16.2
- net FB: now also R15.1, U1.6 (FB); no longer C16.1, R10.1, R11.1, R12.1, R13.1
- net HO: now also Q1.12 (HI), U1.13 (HO)
- net LO: now also Q1.13 (LI), U1.11 (LO)
- net PG: now also U1.17 (PG_SYNCOUT)
- net PGND: now also C16.2, NT1.2, C14.1, C15.1, C17.2, C18.2, C24.2, C25.2, C26.2, C27.2, C28.2, C30.2, C31.2, C33.2, C34.2, C35.2, C36.2, C37.2, C38.2, C39.2, C40.2, C5.2, C7.2, C9.2, Q1.15 (AGND), Q1.17, Q1.6, U1.1 (NC), U1.10 (PGND), U1.14 (SW), U1.16 (VCCX), U1.2 (NC), U1.22 (NC), U1.23 (NC), U1.24 (NC), U1.25 (EP); no longer C4.2, NT1.1
- net RT: now also R2.1, U1.4 (RT); no longer R5.1
- net SW: now also Q1.5
- net U1_EN: now also R3.2, R4.1, U1.19 (EN); no longer R2.2, R3.1
- net U1_VIN: now also U1.12 (VIN)
- net VCC: now also C14.2, C15.2, C5.1, Q1.14 (VCC), U1.9 (VCC)
- net VIN: now also C16.1, C20.1, C21.1, C22.1, R3.1, C17.1, C18.1, C24.1, C27.1, C31.1, C33.1, C34.1, C7.1, Q1.7; no longer C4.1, R2.1
- net VOUT: now also R12.1, C19.1, C25.1, C26.1, C28.1, C30.1, C35.1, C36.1, C37.1, C38.1, C39.1, C40.1, U1.21 (VOUT); no longer C20.1, C21.1, C22.1, L1.2
- net JP_CFG2 renamed FB_RD
- net FB_RD: now also R13.1, R15.2
- new net: Q1.1, Q1.16, Q1.2, Q1.3, Q1.4, Q1.8, Q1.9
- new net CB: C9.1, U1.15 (CBOOT)
- new net CNFG: R5.1, U1.3 (CNFG)
- new net COMP_RC: C4.1, R1.2
- new net HB: C12.2, Q1.10 (HB)
- new net HS: Q1.11 (HS), R8.2
- new net HSB_RC: C12.1, R8.1
- new net ISNS: C19.2, R9.2, U1.20 (ISNS+)
- new net L_OUT: L1.2, R10.1, R11.1, R9.1
- new net VDDA: C1.1, R7.2, U1.8 (VDDA)
- no-connect marks 1 -> 0
Other:
- note added: "12V 10A OUT"
- note added: "DRSS ON"
- note added: "FPWM ONLY!"
- note added: "UVLO Enable @ 37.0V Disable @ 35.0V"
- note added: "derated 13.3uF @ 25V derated 6.3uF @ 50V"
- note added: "derated 75.0uF + 92uF @ 5V derated 36.3uF + 92uF @ 12V"
- note added: "f_{SW} = 450kHz"
- note removed: "5.1V 8A OUT"
- note removed: "Both 12V"
- note removed: "CHANGE"
- note removed: "Config 7.4V"
- note removed: "Config 9.6V"
- note removed: "DEM"
- note removed: "Default 5V"
- note removed: "FCCM"
- note removed: "I_{LIM} = 10.2A @ 5V I_{LIM} = 11.6A @ 12V"
- note removed: "LC pole f_{o} = 5.1kHz @ 5V f_{o} = 6.0kHz @ 12V Inductor Ripple ΔI_{L} = 29% @ 5V ΔI_{L} = 57% @ 12V"
- note removed: "UVLO Enable @ 15.0V Disable @ 13.5V"
- note removed: "derated 15.8uF @ 25V derated 7.6uF @ 50V"
- note removed: "derated 75.0uF + 100uF @ 5V derated 36.3uF + 100uF @ 12V"
- note removed: "f_{SW} = 420kHz"
- note removed: "f_{z1} = 4.8kHz f_{p1} = 48.0kHz"
- note removed: "f_{z2} = 3.4kHz f_{p2} = 1.03MHz"
- note removed: "t_{SS} = 4ms"
- moved on the sheet: C10, C11, C13, C23, C29, C3, C32, C6, C8, D1, D2, J1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
